File: kicad/3320-VCF.kicad_pcb (KiCad board)
At the start: 2 copper layers, 63.5 x 112.3 mm, 63 parts, among them J1 Sig In, J2 Sig Out, J3 FreqCv, J4 ResCv, J5 EuroPower_JST_3P, J6 EURO_PWR_16P, J7 Main, J8 Ctrl, U1 TL072, U2 AS3320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

Commit message: updated pcb revision 0.1.0
Parts:
- added H1: MountingHole_Pad, DIYSynthMNL:MountingHole_M3_Standoff_Pad, F.Cu at (168.1, 54.9)
- added H2: MountingHole_Pad, DIYSynthMNL:MountingHole_M3_Standoff_Pad, F.Cu at (220.5, 54.9)
- C12, C9: footprint DIYSynthMNL:CP_Radial_D4.0mm_P1.50mm -> DIYSynthMNL:CP_Radial_D5.0mm_P2.50mm
Routing:
- net -12V: track 126.3 -> 128.0 mm
- net /3320_Main_Board/3320_IN2: track 25.5 -> 27.2 mm
- net +12V: track 122.3 -> 123.2 mm
- net GND: vias 0 -> 104
- net /3320_Control_Board/CB_GND: vias 0 -> 84
- added copper zone on F.Cu, net /3320_Control_Board/CB_GND
Other:
- board text added: "3320 LP VCF"
- board text added: "3320 Low Pass VCF"
- board text added: "Freq"
- board text added: "FreqCvAmt"
- board text added: "Res"
- board text added: "ResCvAmt"
- board text added: "WayWayWay"
- board text added: "fCvG"
- board text added: "oAmp"
- board text added: "rCvG"
- board text added: "rev 0.1.0"

Commit message: updated pcb rev 0.1.0
Parts:
- added A: Board, PCM_kikit:Board, F.Cu at (162.6, 32.0)
- added B: Board, PCM_kikit:Board, F.Cu at (195.6, 32.0)
- U1: footprint DIYSynthMNL:DIP-8_W7.62mm_LongPads -> Package_DIP:DIP-8_W7.62mm_Socket_LongPads
- U2: footprint DIYSynthMNL:DIP-18_W7.62mm_LongPads -> Package_DIP:DIP-18_W7.62mm_Socket_LongPads
- U3: footprint DIYSynthMNL:DIP-14_W7.62mm_LongPads -> Package_DIP:DIP-14_W7.62mm_Socket_LongPads
- moved R22 3.08 mm to (188.0, 54.4)
- moved C8 1.78 mm to (184.4, 50.0)
- moved C4 0.76 mm to (171.2, 42.4)
- moved C7 0.76 mm to (184.4, 46.5)
- moved C11 0.39 mm to (171.4, 65.8)
- moved C3 0.26 mm to (171.2, 45.5)
- moved R9 0.25 mm to (181.4, 59.2)
Routing:
- net -12V: track 128.0 -> 124.7 mm
- net Net-(U2-VEE): track 7.59 -> 9.25 mm
- net /3320_Main_Board/3320_Out4: track 18.2 -> 17.4 mm
- net +12V: track 123.2 -> 123.8 mm
- net /3320_Main_Board/3320_IN2: track 27.2 -> 27.7 mm
